Commit message: [FIX] Lift L/RJ6 restrictions

File: urdf/robot_v4.xacro (robot description, xacro)
@@ -384,5 +384,5 @@
   <child link="left_hand_1"/>
   <axis xyz="-0.0 1.0 0.0"/>
-  <limit upper="0.0" lower="-1.570796" effort="100" velocity="100"/>
+  <limit upper="1.570796" lower="-1.570796" effort="100" velocity="100"/>
 </joint>
 <joint name="LJ7" type="revolute">
@@ -440,5 +440,5 @@
   <child link="right_hand_1"/>
   <axis xyz="0.0 -1.0 0.0"/>
-  <limit upper="0.0" lower="-1.570796" effort="100" velocity="100"/>
+  <limit upper="1.570796" lower="-1.570796" effort="100" velocity="100"/>
 </joint>
 <joint name="RJ7" type="revolute">
